File: hardware/BREAD_Slice.kicad_sch (KiCad schematic)
At the start: 15 parts, among them J1 Conn_01x10_Female, U1 AP63205

Commit message: updated docs
Connections:
- net DO_out: now reaches A1.19 (A0)
- no-connect marks 22 -> 21
Other:
- added sheet DO Amplifier (do_amp.kicad_sch)
