File: hardware/BREAD_Slice.kicad_pcb (KiCad board)
At the start: 2 copper layers, 70 x 100 mm, 28 parts, among them IC1 TP5551-SR, J1 Conn_01x10_Female, J2 031-5431-1010, U1 AP63205, U2 XC6206PxxxMR

Commit message: fix(hw): re-point stale library nicknames
These parts exist in KiCad-Master-Lib; the boards referenced libraries that no
longer exist (kml-custom, KML-Custom, and SparkFun libraries that never
contained the part) or names the library has since changed.

KiCad embeds footprint geometry in the .kicad_pcb, so the boards rendered and
fabricated correctly and the rot stayed invisible -- it only surfaces on
update-from-library, or when a generator tries to resolve a nickname.

Nickname/name only. No geometry is changed:

  SparkFun-DiscreteSemi:AP63205 -> KMLib_IC_Power:AP63205WU-7_Buck_Regulator
  SparkFun-LED:WS2812-5050-4PIN -> KMLib_IC_SMD:WS2812-5050-4PIN
  kml-custom:03154311010 -> KMLib_Connectors:03154311010
  kml-custom:SOIC127P600X175-8N -> KMLib_IC_SMD:SOIC127P600X175-8N
  kml-custom:TP5551-SR -> KMLib_IC_Analog:TP5551-SR_Chopper_Amplifier
  kml-custom:Thermal Pad -> KMLib_Mounting:Thermal_Pad

Only references that failed to resolve were touched. Generic parts (<=4 pins)
and KiCad *-rescue libraries are deliberately excluded: fingerprint matching
cannot distinguish a 2-pin resistor from a 2-pin capacitor, so those are being
done by hand.
Parts:
- D1: footprint SparkFun-LED:WS2812-5050-4PIN -> KMLib_IC_SMD:WS2812-5050-4PIN
- HS1: footprint kml-custom:Thermal Pad -> KMLib_Mounting:Thermal_Pad
- IC1: footprint kml-custom:SOIC127P600X175-8N -> KMLib_IC_SMD:SOIC127P600X175-8N
- J2: footprint kml-custom:03154311010 -> KMLib_Connectors:03154311010
Changed lines of the file:
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@@
 		)
 	)
-	(footprint "kml-custom:SOIC127P600X175-8N"
+	(footprint "KMLib_IC_SMD:SOIC127P600X175-8N"
 		(layer "F.Cu")
 		(at 167.6 81.365 180)
@@
 		)
 	)
-	(footprint "SparkFun-LED:WS2812-5050-4PIN"
+	(footprint "KMLib_IC_SMD:WS2812-5050-4PIN"
 		(locked yes)
 		(layer "F.Cu")
@@
 		(embedded_fonts no)
 	)
-	(footprint "kml-custom:03154311010"
+	(footprint "KMLib_Connectors:03154311010"
 		(layer "F.Cu")
 		(at 180 80.725 -90)
@@
 		)
 	)
-	(footprint "kml-custom:Thermal Pad"
+	(footprint "KMLib_Mounting:Thermal_Pad"
 		(layer "F.Cu")
 		(at 131.8 121.45)
